Commit message: navigation路径规划

File: src/fishbot_description/urdf/fishbot/base.urdf.xacro (robot description, xacro)
@@ -13,5 +13,5 @@
                 <origin xyz="0 0 0.0" rpy="0 0 0" />
                 <geometry>
-                    <cylinder length="${length}" radius="${length}" />
+                    <cylinder length="${length}" radius="${radius}" />
                 </geometry>
                 <material name="blue">
@@ -22,5 +22,5 @@
                 <origin xyz="0 0 0.0" rpy="0 0 0" />
                 <geometry>
-                    <cylinder length="${length}" radius="${length}" />
+                    <cylinder length="${length}" radius="${radius}" />
                 </geometry>
                 <material name="blue">
